File: Electronics/Rev 2.sch (EAGLE design)
At the start: 52 parts, among them Q1 3STF1640, Q10 3STF1640, Q11 MMBT3904, Q12 DMN601K, Q13 MMBT3904, Q2 DMN601K, Q3 MMBT3904, Q4 3STF1640, Q5 MMBT3904, Q6 DMN601K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

Commit message: Layed out the rev 2 board
Parts:
- removed C5: 0.1uF, Control Cluster Rocket:CAPACITOR0805
Connections:
- net +3V3: no longer C5.P$2
- net DETECT_1: now also U1.BCM_24; no longer U1.BCM_17
- net DETECT_2: now also U1.BCM_12; no longer U1.BCM_18
- net DETECT_3: now also U1.BCM_26; no longer U1.BCM_19
- net DETECT_4: now also U1.BCM_13; no longer U1.BCM_20
- net FIRE_1: now also U1.BCM_23; no longer U1.BCM_6
- net FIRE_2: now also U1.BCM_25; no longer U1.BCM_12
- net FIRE_3: now also U1.BCM_21; no longer U1.BCM_13
- net FIRE_4: now also U1.BCM_19; no longer U1.BCM_16
- net GND: no longer C5.P$1
- net INT1: now also U1.BCM_17; no longer U1.BCM_4
- net INT2: now also U1.BCM_4; no longer U1.BCM_5
- net SPEAKER: now also U1.BCM_18; no longer U1.BCM_21
Changed lines of the file:
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@@
 <part name="GND6" library="Control Cluster Rocket" deviceset="GND" device=""/>
 <part name="C4" library="Control Cluster Rocket" deviceset="CAPACITOR" device="0805" value="0.1uF"/>
-<part name="C5" library="Control Cluster Rocket" deviceset="CAPACITOR" device="0805" value="0.1uF"/>
 <part name="P+8" library="Control Cluster Rocket" deviceset="+3V3" device=""/>
 <part name="GND7" library="Control Cluster Rocket" deviceset="GND" device=""/>
@@
 <net name="INT1" class="0">
 <segment>
+<pinref part="U1" gate="G$1" pin="BCM_17"/>
+<wire x1="81.28" y1="58.42" x2="96.52" y2="73.66" width="0.1524" layer="91"/>
+<label x="83.82" y="73.66" size="1.778" layer="95"/>
+</segment>
+</net>
+<net name="INT2" class="0">
+<segment>
 <pinref part="U1" gate="G$1" pin="BCM_4"/>
-<wire x1="81.28" y1="73.66" x2="96.52" y2="73.66" width="0.1524" layer="91"/>
-<label x="83.82" y="73.66" size="1.778" layer="95"/>
-</segment>
-</net>
-<net name="INT2" class="0">
-<segment>
-<pinref part="U1" gate="G$1" pin="BCM_5"/>
-<wire x1="81.28" y1="71.12" x2="96.52" y2="71.12" width="0.1524" layer="91"/>
+<wire x1="81.28" y1="73.66" x2="96.52" y2="71.12" width="0.1524" layer="91"/>
 <label x="83.82" y="71.12" size="1.778" layer="95"/>
 </segment>
@@
 <net name="FIRE_1" class="0">
 <segment>
-<pinref part="U1" gate="G$1" pin="BCM_6"/>
-<wire x1="81.28" y1="68.58" x2="96.52" y2="68.58" width="0.1524" layer="91"/>
+<pinref part="U1" gate="G$1" pin="BCM_23"/>
+<wire x1="81.28" y1="43.18" x2="96.52" y2="68.58" width="0.1524" layer="91"/>
 <label x="83.82" y="68.58" size="1.778" layer="95"/>
 </segment>
@@
 <net name="FIRE_2" class="0">
 <segment>
+<pinref part="U1" gate="G$1" pin="BCM_25"/>
+<wire x1="81.28" y1="38.1" x2="96.52" y2="66.04" width="0.1524" layer="91"/>
+<label x="83.82" y="66.04" size="1.778" layer="95"/>
+</segment>
+</net>
+<net name="FIRE_3" class="0">
+<segment>
+<pinref part="U1" gate="G$1" pin="BCM_21"/>
+<wire x1="81.28" y1="48.26" x2="96.52" y2="63.5" width="0.1524" layer="91"/>
+<label x="83.82" y="63.5" size="1.778" layer="95"/>
+</segment>
+</net>
+<net name="FIRE_4" class="0">
+<segment>
+<pinref part="U1" gate="G$1" pin="BCM_19"/>
+<wire x1="81.28" y1="53.34" x2="96.52" y2="60.96" width="0.1524" layer="91"/>
+<label x="83.82" y="60.96" size="1.778" layer="95"/>
+</segment>
+</net>
+<net name="DETECT_1" class="0">
+<segment>
+<pinref part="U1" gate="G$1" pin="BCM_24"/>
+<wire x1="81.28" y1="40.64" x2="96.52" y2="58.42" width="0.1524" layer="91"/>
+<label x="83.82" y="58.42" size="1.778" layer="95"/>
+</segment>
+</net>
+<net name="DETECT_2" class="0">
+<segment>
 <pinref part="U1" gate="G$1" pin="BCM_12"/>
-<wire x1="81.28" y1="66.04" x2="96.52" y2="66.04" width="0.1524" layer="91"/>
-<label x="83.82" y="66.04" size="1.778" layer="95"/>
-</segment>
-</net>
-<net name="FIRE_3" class="0">
+<wire x1="81.28" y1="66.04" x2="96.52" y2="55.88" width="0.1524" layer="91"/>
+<label x="83.82" y="55.88" size="1.778" layer="95"/>
+</segment>
+</net>
+<net name="DETECT_3" class="0">
+<segment>
+<pinref part="U1" gate="G$1" pin="BCM_26"/>
+<wire x1="81.28" y1="35.56" x2="96.52" y2="53.34" width="0.1524" layer="91"/>
+<label x="83.82" y="53.34" size="1.778" layer="95"/>
+</segment>
+</net>
+<net name="DETECT_4" class="0">
 <segment>
 <pinref part="U1" gate="G$1" pin="BCM_13"/>
-<wire x1="81.28" y1="63.5" x2="96.52" y2="63.5" width="0.1524" layer="91"/>
-<label x="83.82" y="63.5" size="1.778" layer="95"/>
-</segment>
-</net>
-<net name="FIRE_4" class="0">
-<segment>
-<pinref part="U1" gate="G$1" pin="BCM_16"/>
-<wire x1="81.28" y1="60.96" x2="96.52" y2="60.96" width="0.1524" layer="91"/>
-<label x="83.82" y="60.96" size="1.778" layer="95"/>
-</segment>
-</net>
-<net name="DETECT_1" class="0">
-<segment>
-<pinref part="U1" gate="G$1" pin="BCM_17"/>
-<wire x1="81.28" y1="58.42" x2="96.52" y2="58.42" width="0.1524" layer="91"/>
-<label x="83.82" y="58.42" size="1.778" layer="95"/>
-</segment>
-</net>
-<net name="DETECT_2" class="0">
+<wire x1="81.28" y1="63.5" x2="96.52" y2="50.8" width="0.1524" layer="91"/>
+<label x="83.82" y="50.8" size="1.778" layer="95"/>
+</segment>
+</net>
+<net name="SPEAKER" class="0">
 <segment>
 <pinref part="U1" gate="G$1" pin="BCM_18"/>
-<wire x1="81.28" y1="55.88" x2="96.52" y2="55.88" width="0.1524" layer="91"/>
-<label x="83.82" y="55.88" size="1.778" layer="95"/>
-</segment>
-</net>
-<net name="DETECT_3" class="0">
-<segment>
-<pinref part="U1" gate="G$1" pin="BCM_19"/>
-<wire x1="81.28" y1="53.34" x2="96.52" y2="53.34" width="0.1524" layer="91"/>
-<label x="83.82" y="53.34" size="1.778" layer="95"/>
-</segment>
-</net>
-<net name="DETECT_4" class="0">
-<segment>
-<pinref part="U1" gate="G$1" pin="BCM_20"/>
-<wire x1="81.28" y1="50.8" x2="96.52" y2="50.8" width="0.1524" layer="91"/>
-<label x="83.82" y="50.8" size="1.778" layer="95"/>
-</segment>
-</net>
-<net name="SPEAKER" class="0">
-<segment>
-<pinref part="U1" gate="G$1" pin="BCM_21"/>
-<wire x1="81.28" y1="48.26" x2="96.52" y2="48.26" width="0.1524" layer="91"/>
+<wire x1="81.28" y1="55.88" x2="96.52" y2="48.26" width="0.1524" layer="91"/>
 <label x="83.82" y="48.26" size="1.778" layer="95"/>
 </segment>
@@
 <attribute name="VALUE" x="101.6" y="72.39" size="1.778" layer="96" rot="R90" align="bottom-center"/>
 </instance>
-<instance part="C5" gate="G$1" x="106.68" y="68.58" smashed="yes" rot="R90">
-<attribute name="NAME" x="104.14" y="72.39" size="1.778" layer="95" rot="R90" align="bottom-center"/>
-<attribute name="VALUE" x="111.76" y="72.39" size="1.778" layer="96" rot="R90" align="bottom-center"/>
-</instance>
-<instance part="P+8" gate="G$1" x="101.6" y="83.82" smashed="yes">
-<attribute name="VALUE" x="101.6" y="86.36" size="1.778" layer="96" rot="R180" align="bottom-center"/>
-</instance>
-<instance part="GND7" gate="1" x="101.6" y="60.96" smashed="yes"/>
+<instance part="P+8" gate="G$1" x="96.52" y="81.28" smashed="yes">
+<attribute name="VALUE" x="96.52" y="83.82" size="1.778" layer="96" rot="R180" align="bottom-center"/>
+</instance>
+<instance part="GND7" gate="1" x="96.52" y="63.5" smashed="yes"/>
 <instance part="R1" gate="G$1" x="35.56" y="58.42" smashed="yes" rot="R90">
 <attribute name="NAME" x="33.02" y="66.04" size="1.778" layer="95" rot="R90" align="bottom-center"/>
@@
 <pinref part="C4" gate="G$1" pin="P$2"/>
 <wire x1="96.52" y1="76.2" x2="96.52" y2="78.74" width="0.1524" layer="91"/>
-<wire x1="96.52" y1="78.74" x2="101.6" y2="78.74" width="0.1524" layer="91"/>
 <pinref part="P+8" gate="G$1" pin="+3V3"/>
-<wire x1="101.6" y1="78.74" x2="101.6" y2="81.28" width="0.1524" layer="91"/>
-<wire x1="101.6" y1="78.74" x2="106.68" y2="78.74" width="0.1524" layer="91"/>
-<junction x="101.6" y="78.74"/>
-<pinref part="C5" gate="G$1" pin="P$2"/>
-<wire x1="106.68" y1="78.74" x2="106.68" y2="76.2" width="0.1524" layer="91"/>
 </segment>
 <segment>
@@
 <segment>
 <pinref part="GND7" gate="1" pin="GND"/>
-<wire x1="101.6" y1="63.5" x2="101.6" y2="66.04" width="0.1524" layer="91"/>
-<pinref part="C5" gate="G$1" pin="P$1"/>
-<wire x1="101.6" y1="66.04" x2="106.68" y2="66.04" width="0.1524" layer="91"/>
-<wire x1="106.68" y1="66.04" x2="106.68" y2="68.58" width="0.1524" layer="91"/>
 <pinref part="C4" gate="G$1" pin="P$1"/>
-<wire x1="101.6" y1="66.04" x2="96.52" y2="66.04" width="0.1524" layer="91"/>
 <wire x1="96.52" y1="66.04" x2="96.52" y2="68.58" width="0.1524" layer="91"/>
-<junction x="101.6" y="66.04"/>
-</segment>
-<segment>
+</segment>
+<segment>
