File: Electronics/Rev 2.brd (EAGLE design)
At the start: 50.8 x 101.6 mm, 51 parts, among them Q1 3STF1640, Q10 3STF1640, Q11 MMBT3904, Q12 DMN601K, Q13 MMBT3904, Q2 DMN601K, Q3 MMBT3904, Q4 3STF1640, Q5 MMBT3904, Q6 DMN601K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

Commit message: Finished electronics
Routing:
- net +3V3: track 117.6 -> 114.8 mm
- net SDA: track 34.7 -> 36.5 mm
- net INT1: track 31.9 -> 32.9 mm
- net SCL: track 40.3 -> 41.1 mm
- net FIRE_3: track 12.4 -> 13.0 mm
- net DETECT_3: track 78.5 -> 79.1 mm
